Commit message: comment changed

File: examples/rsc/chain/robot.urdf (robot description, URDF)
Before this commit: robot 2DrobotArm, 5 links, 4 joints
Links:
- removed link link3
- removed link link4
Joints:
- removed joint link2Tolink3
- removed joint link3Tolink4
- joint link1Tolink2: origin xyz=0 0 -0.34 -> xyz=0 0 -0.50
